Commit message: fix scale

File: urdf/r1.urdf.xacro (robot description, xacro)
@@ -27,5 +27,5 @@
 	    	<visual>
 	    		<geometry>
-	    			<mesh filename="package://aion_r1_description/R1Mesh/wheel.stl" />
+	    			<mesh filename="package://aion_r1_description/R1Mesh/wheel.stl" scale="0.01 0.01 0.01"/>
 				</geometry>
 				<material name="black" />
@@ -81,5 +81,5 @@
       <visual>
         <geometry>
-          <mesh filename="package://aion_r1_description/R1Mesh/antenna.stl" />
+          <mesh filename="package://aion_r1_description/R1Mesh/antenna.stl" scale="0.01 0.01 0.01"/>
         </geometry>
         <material name="black" />
@@ -120,5 +120,5 @@
     <visual>
       <geometry>
-        <mesh filename="package://aion_r1_description/R1Mesh/body.stl" />
+        <mesh filename="package://aion_r1_description/R1Mesh/body.stl" scale="0.01 0.01 0.01" />
       </geometry>
       <material name="gray" />
@@ -151,5 +151,5 @@
     <visual>
       <geometry>
-        <mesh filename="package://aion_r1_description/R1Mesh/top.stl" />
+        <mesh filename="package://aion_r1_description/R1Mesh/top.stl" scale="0.01 0.01 0.01"/>
       </geometry>
       <material name="white" />
@@ -174,5 +174,5 @@
     <visual>
       <geometry>
-        <mesh filename="package://aion_r1_description/R1Mesh/battery.stl" />
+        <mesh filename="package://aion_r1_description/R1Mesh/battery.stl" scale="0.01 0.01 0.01"/>
       </geometry>
       <material name="black" />
@@ -197,5 +197,5 @@
     <visual>
       <geometry>
-        <mesh filename="package://aion_r1_description/R1Mesh/housing.stl" />
+        <mesh filename="package://aion_r1_description/R1Mesh/housing.stl" scale="0.01 0.01 0.01"/>
       </geometry>
       <material name="black" />

Commit message: wip

File: urdf/r1.urdf.xacro (robot description, xacro)
@@ -119,4 +119,7 @@
     </inertial>
     <visual>
+      <origin
+        xyz="0 0 0"
+        rpy="0 0 0" />
       <geometry>
         <mesh filename="package://aion_r1_description/R1Mesh/body.stl" scale="0.01 0.01 0.01" />
