Commit message: fix new r1 description

File: urdf/materials.urdf.xacro (robot description, xacro)
@@ -10,3 +10,6 @@
 		<color rgba="0.9 0.9 0.9 1.0" />
 	</material>
+	<material name="safety_orange">
+		<color rgba="1.0 0.4 0.0 1.0" />
+	</material>
 </robot>

File: urdf/r1.urdf.xacro (robot description, xacro)
@@ -54,5 +54,5 @@
 			type="fixed">
 			<origin
-				xyz="${0.1475 * reflect_x} ${0.16 * reflect_y} 0.0327"
+				xyz="${0.1475 * reflect_x} ${0.16 * reflect_y} -0.0327"
 				rpy="0 0 0" />
 			<parent link="base_link" />
@@ -90,5 +90,5 @@
       type="fixed">
       <origin
-        xyz="-0.1525 ${0.0814 * reflect} 0.0584"
+        xyz="-0.1475 ${0.0814 * reflect} 0.1145"
         rpy="0 0 0" />
       <parent
@@ -205,4 +205,50 @@
     </visual>
   </link>
+  <link
+    name="bridge_link">
+    <inertial>
+      <origin
+        xyz="0 0 0"
+        rpy="0 0 0" />
+      <mass
+        value="0.04" />
+      <inertia
+        ixx="4.349e-05"
+        ixy="0"
+        ixz="-1.89e-06"
+        iyy="4.241e-05"
+        iyz="0"
+        izz="7.779e-05" />
+    </inertial>
+    <visual>
+      <geometry>
+        <mesh filename="package://aion_r1_description/R1Mesh/gpsbridge.stl" scale="0.01 0.01 0.01"/>
+      </geometry>
+      <material name="safety_orange" />
+    </visual>
+  </link>
+  <link
+    name="vlp16_link">
+    <inertial>
+      <origin
+        xyz="0 0 0"
+        rpy="0 0 0" />
+      <mass
+        value="0.04" />
+      <inertia
+        ixx="4.349e-05"
+        ixy="0"
+        ixz="-1.89e-06"
+        iyy="4.241e-05"
+        iyz="0"
+        izz="7.779e-05" />
+    </inertial>
+    <visual>
+      <geometry>
+        <mesh filename="package://aion_r1_description/R1Mesh/VLP16.stl" scale="0.01 0.01 0.01"/>
+      </geometry>
+      <material name="gray" />
+    </visual>
+  </link>
   <!-- Defining model joints. -->
   <joint
@@ -222,4 +268,22 @@
   </joint>
   <joint
+    name="fixed_bridge_joint"
+    type="fixed">
+    <origin
+      xyz="0.0525 0 0.109"
+      rpy="0 0 0" />
+    <parent link="base_link" />
+    <child link="bridge_link" />
+  </joint>
+  <joint
+    name="fixed_vlp16_joint"
+    type="fixed">
+    <origin
+      xyz="0.0927 0 0.2252"
+      rpy="0 0 0" />
+    <parent link="base_link" />
+    <child link="vlp16_link" />
+  </joint>
+  <joint
     name="fixed_battery_joint"
     type="fixed">
@@ -242,5 +306,5 @@
   <!--Front Camera-->
   <sensor_d435 name="camera1" parent="base_link">
-    <origin xyz="0.1880 0 0.0505" rpy="0 0 0"/>
+    <origin xyz="0.1880 0 0" rpy="0 0 0"/>
   </sensor_d435>
   <joint name="gazebo_cam_joint" type="fixed">
